File: PCB/galvanosynth.kicad_pcb (KiCad board)
At the start: 2 copper layers, 127 x 63.5 mm, 81 parts, among them J1 Conn_01x40, U0 L7815, U1 LM358, U2 LM358, U3 LM358, U4 LM358, U5 LM358, U6 LM358, U7 LM358, U8 LM358

Commit message: forgotten
Parts:
- removed G***: LOGO, footprints:logo
- added R1: 68, Resistor_SMD:R_1206_3216Metric, F.Cu at (157.5, 67.3)
- added RL1: 10, Resistor_SMD:R_1206_3216Metric, F.Cu at (69.8, 113.0)
- added RL2: 10, Resistor_SMD:R_1206_3216Metric, F.Cu at (82.5, 113.0)
- added RL3: 10, Resistor_SMD:R_1206_3216Metric, F.Cu at (95.2, 113.0)
- added RL4: 10, Resistor_SMD:R_1206_3216Metric, F.Cu at (108.0, 113.0)
- added RL5: 10, Resistor_SMD:R_1206_3216Metric, F.Cu at (120.7, 113.0)
- added RL6: 10, Resistor_SMD:R_1206_3216Metric, F.Cu at (133.3, 113.0)
- added RL7: 10, Resistor_SMD:R_1206_3216Metric, F.Cu at (146.1, 113.0)
- added RL8: 10, Resistor_SMD:R_1206_3216Metric, F.Cu at (158.8, 113.0)
- C1: value 10uF -> 100uF
- R0: value R_US -> 10k; footprint Resistor_THT:R_Axial_DIN0207_L6.3mm_D2.5mm_P7.62mm_Horizontal -> Resistor_SMD:R_1206_3216Metric
- RF1, RF2, RF3, RF4, RF5, RF6, RF7, RF8, RG1, RG2, RG3, RG4, RG5, RG6, RG7, RG8: value 10k -> 100k
- RV0: value 10k -> 1k
- moved R0 1.40 mm to (157.5, 72.3)
Connections:
- RV0 pad 3: GND -> Net-(R1-Pad1)
- RV1 pad 1: GND -> Net-(RL1-Pad2)
- RV2 pad 1: GND -> Net-(RL2-Pad2)
- RV3 pad 1: GND -> Net-(RL3-Pad2)
- RV4 pad 1: GND -> Net-(RL4-Pad2)
- RV5 pad 1: GND -> Net-(RL5-Pad2)
- RV6 pad 1: GND -> Net-(RL6-Pad2)
- RV7 pad 1: GND -> Net-(RL7-Pad2)
- RV8 pad 1: GND -> Net-(RL8-Pad2)
Routing:
- net +15V: track 566.8 -> 556.7 mm, vias 0 -> 1
- net Net-(RL7-Pad2): track 0.00 -> 5.48 mm
- net Net-(RL5-Pad2): track 0.00 -> 5.48 mm
- net Net-(RL2-Pad2): track 0.00 -> 5.48 mm
- net Net-(RL1-Pad2): track 0.00 -> 5.48 mm
- net Net-(RL4-Pad2): track 0.00 -> 5.48 mm
- net Net-(RL8-Pad2): track 0.00 -> 5.48 mm
- net Net-(RL3-Pad2): track 0.00 -> 5.48 mm
- net Net-(RL6-Pad2): track 0.00 -> 5.48 mm
- net Net-(R1-Pad1): track 0.00 -> 5.13 mm
- net /1/RETURN: track 43.0 -> 38.3 mm
- net /8/RETURN: track 43.0 -> 38.4 mm
- net /2/RETURN: track 43.0 -> 38.4 mm
- net /4/RETURN: track 43.0 -> 38.4 mm
- net /3/RETURN: track 43.0 -> 38.4 mm
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Other:
- board text added: "REVISION 4.1.1 MARCH 2020"
- board text removed: "GALVANOSYNTH"
- board text removed: "REVISION 4.1.0 JANUARY 2020"
