File: daugher/daughter.kicad_pcb (KiCad board)
At the start: 2 copper layers, 127 x 50.8 mm, 36 parts, among them J1 Conn_01x40

Commit message: forgotten
Parts:
- added REF**: MountingHole_3.2mm_M3, MountingHole:MountingHole_3.2mm_M3, F.Cu at (172.7, 106.0)
- added REF**: MountingHole_3.2mm_M3, MountingHole:MountingHole_3.2mm_M3, F.Cu at (55.9, 106.0)
- moved G*** 2.54 mm to (171.4, 92.7)
Other:
- board text added: "FRONT PANEL REVISION 1.3.1 MARCH 2020"
- board text removed: "FRONT PANEL REVISION 1.2.0 JANUARY 2020"
