File: galvanosyth/front-panel-pcb/kicad/front-panel.kicad_pcb (KiCad board)
At the start: 2 copper layers, 127 x 50.8 mm, 38 parts, among them J1 Conn_01x40

Commit message: galvo front panel organize
Other:
- rule pad_to_mask_clearance: 0.051 -> 0
