File: potentiosynth/front-panel-pcb/kicad/front-panel.sch (KiCad schematic (older format))
At the start: 35 parts, among them J1 Conn_01x40

Commit message: first draft front panel
Parts:
- added D10, D9: LED, Diode_SMD:D_1206_3216Metric, symbol Device:LED
- added J_WRK1, J_WRK2, J_WRK3, J_WRK4, J_WRK5, J_WRK6, J_WRK7, J_WRK8: Conn_01x01, Connector:Banana_Jack_1Pin, symbol Connector_Generic:Conn_01x01
- added R10, R9: 1k, Resistor_SMD:R_1206_3216Metric, symbol Device:R_US
- added SW1: SW_SPDT, Connector_PinHeader_2.54mm:PinHeader_1x03_P2.54mm_Horizontal, symbol Switch:SW_SPDT
- renumbered J_ANO1 to J_COU1, J_ANO2 to J_COU2, J_ANO3 to J_COU3, J_ANO4 to J_COU4, J_ANO5 to J_COU5, J_ANO6 to J_COU6, J_ANO7 to J_COU7, J_ANO8 to J_COU8, J_CAT1 to J_REF1, J_CAT2 to J_REF2, J_CAT3 to J_REF3, J_CAT4 to J_REF4, J_CAT5 to J_REF5, J_CAT6 to J_REF6, J_CAT7 to J_REF7, J_CAT8 to J_REF8
Connections:
- net +15V: now also R9.1, SW1.3 (C)
- net GND: now also D10.1 (K), SW1.1 (A)
- new net: D9.2 (A), R9.2
- new net: D10.2 (A), R10.2
- new net WORKING: D9.1 (K), J_WRK1.1 (Pin_1), J_WRK2.1 (Pin_1), J_WRK3.1 (Pin_1), J_WRK4.1 (Pin_1), J_WRK5.1 (Pin_1), J_WRK6.1 (Pin_1), J_WRK7.1 (Pin_1), J_WRK8.1 (Pin_1), R10.1, SW1.2 (B)
Other:
- note added: "LIGHTS WHEN\nWORKING +15V\nOXIDATION"
- note added: "LIGHTS WHEN\nWORKING GROUND\nREDUCTION"
