File: potentiosynth/driver-pcb/kicad/potentiosynth.kicad_pcb (KiCad board)
At the start: 2 copper layers, 127 x 63.5 mm, 70 parts, among them J1 Conn_01x40, U0 R-7815-0.5, U1 TLV9154IDR, U2 TLV9154IDR, U3 TLV9154IDR, U4 TLV9154IDR, U5 TLV9154IDR, U6 TLV9154IDR, U7 TLV9154IDR, U8 TLV9154IDR

Commit message: resistor net
Parts:
- removed R+1, R+2, R+3, R+4, R+5, R+6, R+7, R+8, R-1, R-2, R-3, R-4, R-5, R-6, R-7, R-8: 1k, Resistor_SMD:R_1206_3216Metric
- removed RF1, RF2, RF3, RF4, RF5, RF6, RF7, RF8, RG1, RG2, RG3, RG4, RG5, RG6, RG7, RG8: 100k, Resistor_SMD:R_1206_3216Metric
- added QEN1: 2N70002K, Package_TO_SOT_SMD:SOT-23_Handsoldering, F.Cu at (62.5, 108.2)
- added QEN2: 2N70002K, Package_TO_SOT_SMD:SOT-23_Handsoldering, F.Cu at (85.1, 91.4)
- added QEN3: 2N70002K, Package_TO_SOT_SMD:SOT-23_Handsoldering, F.Cu at (94.5, 144.3)
- added QEN4: 2N70002K, Package_TO_SOT_SMD:SOT-23_Handsoldering, F.Cu at (110.2, 144.7)
- added QEN5: 2N70002K, Package_TO_SOT_SMD:SOT-23_Handsoldering, F.Cu at (125.5, 144.5)
- added QEN6: 2N70002K, Package_TO_SOT_SMD:SOT-23_Handsoldering, F.Cu at (142.3, 145.8)
- added QEN7: 2N70002K, Package_TO_SOT_SMD:SOT-23_Handsoldering, F.Cu at (159.0, 146.3)
- added QEN8: 2N70002K, Package_TO_SOT_SMD:SOT-23_Handsoldering, F.Cu at (175.8, 148.6)
- added RNH1: 100k, footprints:CAY16-104J4LF, F.Cu at (67.8, 85.0)
- added RNH2: 100k, footprints:CAY16-104J4LF, F.Cu at (85.7, 97.8)
- added RNH3: 100k, footprints:CAY16-104J4LF, F.Cu at (104.2, 144.9)
- added RNH4: 100k, footprints:CAY16-104J4LF, F.Cu at (119.9, 145.4)
- added RNH5: 100k, footprints:CAY16-104J4LF, F.Cu at (130.9, 145.2)
- added RNH6: 100k, footprints:CAY16-104J4LF, F.Cu at (147.7, 146.5)
- added RNH7: 100k, footprints:CAY16-104J4LF, F.Cu at (164.4, 146.9)
- added RNH8: 100k, footprints:CAY16-104J4LF, F.Cu at (181.2, 149.2)
- added RNL1: 1k, footprints:CAY16-104J4LF, F.Cu at (72.1, 85.0)
- added RNL2: 1k, footprints:CAY16-104J4LF, F.Cu at (79.4, 97.8)
- added RNL3: 1k, footprints:CAY16-104J4LF, F.Cu at (99.9, 144.9)
- added RNL4: 1k, footprints:CAY16-104J4LF, F.Cu at (115.6, 145.4)
- added RNL5: 1k, footprints:CAY16-104J4LF, F.Cu at (135.1, 145.2)
- added RNL6: 1k, footprints:CAY16-104J4LF, F.Cu at (151.9, 146.5)
- added RNL7: 1k, footprints:CAY16-104J4LF, F.Cu at (168.7, 146.9)
- added RNL8: 1k, footprints:CAY16-104J4LF, F.Cu at (185.5, 149.2)
- RV1, RV2, RV3, RV4, RV5, RV6, RV7, RV8: value R_POT_US -> 2k
- moved QEP2 18.0 mm to (80.0, 91.4), turned to 90 degrees
- moved U2 5.08 mm to (82.5, 105.4), turned to 270 degrees
- renumbered QE1 to QEP1, QE2 to QEP2, QE3 to QEP3, QE4 to QEP4, QE5 to QEP5, QE6 to QEP6, QE7 to QEP7, QE8 to QEP8
Connections:
- U1 pad 1: (no net) -> Net-(QEN1-Pad1)
- U1 pad 2: (no net) -> Net-(RNH1-Pad2)
- U1 pad 3: (no net) -> Net-(RNH1-Pad4)
- U2 pad 1: (no net) -> Net-(QEN2-Pad1)
- U2 pad 2: (no net) -> Net-(RNH2-Pad2)
- U2 pad 3: (no net) -> Net-(RNH2-Pad4)
- U3 pad 1: (no net) -> Net-(QEN3-Pad1)
- U3 pad 2: (no net) -> Net-(RNH3-Pad2)
- U3 pad 3: (no net) -> Net-(RNH3-Pad4)
- U4 pad 1: (no net) -> Net-(QEN4-Pad1)
- U4 pad 2: (no net) -> Net-(RNH4-Pad2)
- U4 pad 3: (no net) -> Net-(RNH4-Pad4)
- U5 pad 1: (no net) -> Net-(QEN5-Pad1)
- U5 pad 2: (no net) -> Net-(RNH5-Pad2)
- U5 pad 3: (no net) -> Net-(RNH5-Pad4)
- U6 pad 1: (no net) -> Net-(QEN6-Pad1)
- U6 pad 2: (no net) -> Net-(RNH6-Pad2)
- U6 pad 3: (no net) -> Net-(RNH6-Pad4)
- U7 pad 1: (no net) -> Net-(QEN7-Pad1)
- U7 pad 2: (no net) -> Net-(RNH7-Pad2)
- U7 pad 3: (no net) -> Net-(RNH7-Pad4)
- U8 pad 1: (no net) -> Net-(QEN8-Pad1)
- U8 pad 2: (no net) -> Net-(RNH8-Pad2)
- U8 pad 3: (no net) -> Net-(RNH8-Pad4)
Routing:
- net Net-(RNL2-Pad1): track 41.5 -> 0.00 mm, vias 1 -> 0
- net /2/REFERENCE: track 34.4 -> 0.00 mm, vias 1 -> 0
- net /2/COUNTER: track 30.0 -> 0.00 mm, vias 1 -> 0
- net Net-(QEP2-Pad1): track 23.7 -> 0.00 mm
- net Net-(QEN2-Pad1): track 0.00 -> 21.1 mm
- net GND: track 181.8 -> 163.8 mm
- net Net-(RNL2-Pad2): track 16.7 -> 0.00 mm
- net Net-(RNH2-Pad8): track 15.4 -> 0.03 mm
- net /2/ERROR: track 13.5 -> 0.00 mm
- net Net-(RNH2-Pad3): track 19.9 -> 7.29 mm
- net +15V: track 99.4 -> 91.7 mm, vias 8 -> 7
- net Net-(RNH8-Pad3): track 19.9 -> 12.4 mm
- net Net-(RNH7-Pad3): track 19.9 -> 12.4 mm
- net Net-(RNH5-Pad3): track 19.9 -> 12.4 mm
- net Net-(RNH4-Pad3): track 19.9 -> 12.4 mm
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
Commit message: potentiosynth driver revC
Parts:
- added C1: C, Capacitor_SMD:C_1206_3216Metric_Pad1.33x1.80mm_HandSolder, F.Cu at (70.8, 111.8)
- added C102: 330nF, Capacitor_SMD:C_1206_3216Metric_Pad1.33x1.80mm_HandSolder, F.Cu at (116.8, 66.0)
- added C3: C, Capacitor_SMD:C_1206_3216Metric_Pad1.33x1.80mm_HandSolder, F.Cu at (96.2, 111.8)
- added C4: C, Capacitor_SMD:C_1206_3216Metric_Pad1.33x1.80mm_HandSolder, F.Cu at (108.9, 111.8)
- added C5: C, Capacitor_SMD:C_1206_3216Metric_Pad1.33x1.80mm_HandSolder, F.Cu at (121.6, 111.8)
- added C6: C, Capacitor_SMD:C_1206_3216Metric_Pad1.33x1.80mm_HandSolder, F.Cu at (134.3, 111.8)
- added C7: C, Capacitor_SMD:C_1206_3216Metric_Pad1.33x1.80mm_HandSolder, F.Cu at (147.0, 111.8)
- added C8: C, Capacitor_SMD:C_1206_3216Metric_Pad1.33x1.80mm_HandSolder, F.Cu at (159.7, 111.8)
- added REF**: OSHW-Logo2_14.6x12mm_SilkScreen, Symbol:OSHW-Logo2_14.6x12mm_SilkScreen, B.Cu at (114.3, 78.1)
- C103: renamed from C3; footprint Capacitor_THT:CP_Radial_Tantal_D7.0mm_P2.50mm -> Capacitor_SMD:C_1206_3216Metric_Pad1.33x1.80mm_HandSolder
- C2: value 330nF -> C; footprint Capacitor_THT:CP_Radial_Tantal_D7.0mm_P2.50mm -> Capacitor_SMD:C_1206_3216Metric_Pad1.33x1.80mm_HandSolder
- moved RNL8 59.5 mm to (155.6, 97.8), turned to 90 degrees
- moved QEN8 59.0 mm to (161.3, 91.4), turned to 90 degrees
- moved QEN7 55.8 mm to (148.6, 91.4), turned to 90 degrees
- moved RNL7 55.5 mm to (142.9, 97.8), turned to 90 degrees
- moved RNH8 54.9 mm to (161.9, 97.8), turned to 90 degrees
- moved QEN6 54.7 mm to (135.9, 91.4), turned to 90 degrees
- moved RNL6 53.3 mm to (130.2, 97.8), turned to 90 degrees
- moved QEN4 53.3 mm to (110.5, 91.4), turned to 90 degrees
- moved QEN5 53.1 mm to (123.2, 91.4), turned to 90 degrees
- moved QEN3 52.9 mm to (97.8, 91.4), turned to 90 degrees
- moved RNH7 51.4 mm to (149.2, 97.8), turned to 90 degrees
- moved RNL5 50.6 mm to (117.5, 97.8), turned to 90 degrees
- moved RNH6 49.9 mm to (136.5, 97.8), turned to 90 degrees
- moved RNL4 48.8 mm to (104.8, 97.8), turned to 90 degrees
- moved C2 48.8 mm to (83.5, 111.8), turned to 180 degrees
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- renumbered C1 to C101
Connections:
- C101 pad 1: Net-(C1-Pad1) -> Net-(C101-Pad1)
- C2 pad 1: Net-(C1-Pad1) -> /2/REFERENCE
- F1 pad 2: Net-(C1-Pad1) -> Net-(C101-Pad1)
- RNL1 pad 2: Net-(RNL1-Pad2) -> Net-(RNL1-Pad1)
- RNL1 pad 3: Net-(RNL1-Pad2) -> Net-(RNL1-Pad3)
- RNL1 pad 4: Net-(RNL1-Pad1) -> Net-(RNL1-Pad3)
- RNL1 pad 5: Net-(RNH1-Pad2) -> Net-(RNH1-Pad8)
- RNL1 pad 7: Net-(RNH1-Pad8) -> Net-(RNH1-Pad2)
- RNL2 pad 2: Net-(RNL2-Pad2) -> Net-(RNL2-Pad1)
- RNL2 pad 3: Net-(RNL2-Pad2) -> Net-(RNL2-Pad3)
- RNL2 pad 4: Net-(RNL2-Pad1) -> Net-(RNL2-Pad3)
- RNL2 pad 5: Net-(RNH2-Pad2) -> Net-(RNH2-Pad8)
- RNL2 pad 7: Net-(RNH2-Pad8) -> Net-(RNH2-Pad2)
- RNL3 pad 2: Net-(RNL3-Pad2) -> Net-(RNL3-Pad1)
- RNL3 pad 3: Net-(RNL3-Pad2) -> Net-(RNL3-Pad3)
- RNL3 pad 4: Net-(RNL3-Pad1) -> Net-(RNL3-Pad3)
- RNL3 pad 5: Net-(RNH3-Pad2) -> Net-(RNH3-Pad8)
- RNL3 pad 7: Net-(RNH3-Pad8) -> Net-(RNH3-Pad2)
- RNL4 pad 2: Net-(RNL4-Pad2) -> Net-(RNL4-Pad1)
- RNL4 pad 3: Net-(RNL4-Pad2) -> Net-(RNL4-Pad3)
- RNL4 pad 4: Net-(RNL4-Pad1) -> Net-(RNL4-Pad3)
- RNL4 pad 5: Net-(RNH4-Pad2) -> Net-(RNH4-Pad8)
- RNL4 pad 7: Net-(RNH4-Pad8) -> Net-(RNH4-Pad2)
- RNL5 pad 2: Net-(RNL5-Pad2) -> Net-(RNL5-Pad1)
- RNL5 pad 3: Net-(RNL5-Pad2) -> Net-(RNL5-Pad3)
- RNL5 pad 4: Net-(RNL5-Pad1) -> Net-(RNL5-Pad3)
- RNL5 pad 5: Net-(RNH5-Pad2) -> Net-(RNH5-Pad8)
- RNL5 pad 7: Net-(RNH5-Pad8) -> Net-(RNH5-Pad2)
- RNL6 pad 2: Net-(RNL6-Pad2) -> Net-(RNL6-Pad1)
- RNL6 pad 3: Net-(RNL6-Pad2) -> Net-(RNL6-Pad3)
- RNL6 pad 4: Net-(RNL6-Pad1) -> Net-(RNL6-Pad3)
- RNL6 pad 5: Net-(RNH6-Pad2) -> Net-(RNH6-Pad8)
- RNL6 pad 7: Net-(RNH6-Pad8) -> Net-(RNH6-Pad2)
- RNL7 pad 2: Net-(RNL7-Pad2) -> Net-(RNL7-Pad1)
- RNL7 pad 3: Net-(RNL7-Pad2) -> Net-(RNL7-Pad3)
- RNL7 pad 4: Net-(RNL7-Pad1) -> Net-(RNL7-Pad3)
- RNL7 pad 5: Net-(RNH7-Pad2) -> Net-(RNH7-Pad8)
- RNL7 pad 7: Net-(RNH7-Pad8) -> Net-(RNH7-Pad2)
- RNL8 pad 2: Net-(RNL8-Pad2) -> Net-(RNL8-Pad1)
- RNL8 pad 3: Net-(RNL8-Pad2) -> Net-(RNL8-Pad3)
- RNL8 pad 4: Net-(RNL8-Pad1) -> Net-(RNL8-Pad3)
- RNL8 pad 5: Net-(RNH8-Pad2) -> Net-(RNH8-Pad8)
- RNL8 pad 7: Net-(RNH8-Pad8) -> Net-(RNH8-Pad2)
- U0 pad 1: Net-(C1-Pad1) -> Net-(C101-Pad1)
- U1 pad 8: Net-(RNL1-Pad2) -> Net-(RNL1-Pad3)
- U1 pad 9: Net-(RNL1-Pad2) -> Net-(RNL1-Pad3)
- U2 pad 8: Net-(RNL2-Pad2) -> Net-(RNL2-Pad3)
- U2 pad 9: Net-(RNL2-Pad2) -> Net-(RNL2-Pad3)
- U3 pad 8: Net-(RNL3-Pad2) -> Net-(RNL3-Pad3)
- U3 pad 9: Net-(RNL3-Pad2) -> Net-(RNL3-Pad3)
- U4 pad 8: Net-(RNL4-Pad2) -> Net-(RNL4-Pad3)
- U4 pad 9: Net-(RNL4-Pad2) -> Net-(RNL4-Pad3)
- U5 pad 8: Net-(RNL5-Pad2) -> Net-(RNL5-Pad3)
- U5 pad 9: Net-(RNL5-Pad2) -> Net-(RNL5-Pad3)
- U6 pad 8: Net-(RNL6-Pad2) -> Net-(RNL6-Pad3)
- U6 pad 9: Net-(RNL6-Pad2) -> Net-(RNL6-Pad3)
- U7 pad 8: Net-(RNL7-Pad2) -> Net-(RNL7-Pad3)
- U7 pad 9: Net-(RNL7-Pad2) -> Net-(RNL7-Pad3)
- U8 pad 8: Net-(RNL8-Pad2) -> Net-(RNL8-Pad3)
- U8 pad 9: Net-(RNL8-Pad2) -> Net-(RNL8-Pad3)
Routing:
- net GND: track 163.8 -> 1.12 mm
- net /2/ERROR: track 0.00 -> 39.6 mm, vias 0 -> 1
- net +15V: track 91.7 -> 56.8 mm, vias 7 -> 8
- net Net-(RNL2-Pad1): track 0.00 -> 31.6 mm
- net Net-(C101-Pad1): track 0.00 -> 28.5 mm
- net Net-(RNH8-Pad4): track 0.00 -> 27.7 mm, vias 0 -> 2
- net Net-(RNH5-Pad4): track 0.00 -> 27.7 mm, vias 0 -> 2
- net Net-(RNH7-Pad4): track 0.00 -> 27.7 mm, vias 0 -> 2
- net Net-(RNH4-Pad4): track 0.00 -> 27.7 mm, vias 0 -> 2
- net Net-(RNH6-Pad4): track 0.00 -> 27.7 mm, vias 0 -> 2
- net Net-(RNH1-Pad4): track 0.00 -> 27.6 mm, vias 0 -> 2
- net Net-(RNH3-Pad4): track 0.00 -> 27.6 mm, vias 0 -> 2
- net /2/REFERENCE: track 0.00 -> 26.5 mm
- net Net-(QEP2-Pad1): track 0.00 -> 26.1 mm, vias 0 -> 2
- net Net-(C1-Pad1): track 26.1 -> 0.00 mm
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Other:
- net class Default: trace_width 0.508 -> 0.381
- board text added: "18 to 30 V DC CENTER POSITIVE"
- board text added: "POTENTIOSYNTH REVISION C OCTOBER 2021"
- board text added: "https://github.com/ uw-madison-chem-shops/ electrosynth/"
- board text removed: "18 to 30 V"
- board text removed: "POTENTIOSYNTH REVISION B JULY 2021"
